File: glove_eagle/glove.sch (EAGLE design)
At the start: 20 parts, among them U1 BNO055, U2 NRF51822-QFAA-T

Commit message: Added Lab 11 libraries / Started charging circuit
Parts:
- removed C10: 47 nF, rcl:C-USC0402
- removed C11, C8: 100 nF, rcl:C-USC0402
- removed C12: 1.0 uF, rcl:C-USC0603
- removed C4: 1.0 pF, rcl:C-USC0402
- removed C5: 3.9 pF, rcl:C-USC0402
- removed C6: 1.5 pF, rcl:C-USC0402
- removed C7: 4.7 uF, rcl:C-USC0603
- removed C9: 1.0 nF, rcl:C-USC0402
- removed L1: 4.7 nH, passives:INDUCTOR0402
- removed L2, L4, L5: 27 nH, passives:INDUCTOR0402
- removed L3: 3.3 nH, passives:INDUCTOR0402
- removed U2: NRF51822-QFAA-T, NRF51822-QFAA-T:NRF51822-QFAA-T
- removed X1: (no value), crystals:FH1600015
- added A1: FRACTUS-2.4GHZ-FR05-S1-N-0-102, chips:FRACTUS-2.4GHZ-FR05-S1-N-0-102
- added B1: BAL-NRF01D3, chips:BAL-NRF01D3
- added C13, C14: 100 nF, rcl:C-USC0603
- added C15: 120 nF, rcl:C-USC0603
- added C16: 6.8 nF, rcl:C-USC0603
- added C17, C18, C19, C20: 12 pF, passives:CAPACITOR0402_CAP
- added C21: 2.2 nF, passives:CAPACITOR0402_CAP
- added C22, C27: 1.0 nF, passives:CAPACITOR0402_CAP
- added C24: 0.8 pF, passives:CAPACITOR0402_CAP
- added C25: 100 nF, passives:CAPACITOR0402_CAP
- added C28: 47 nF, passives:CAPACITOR0402_CAP
- added C29: 4.7 uF, passives:CAPACITOR0603_CAP
- added C30: 1.0 uF, passives:CAPACITOR0603_CAP
- added J1: MICRO_USB_B_JST_MC5BR3-M404-4S, connector:MICRO_USB_B_JST_MC5BR3-M404-4S
- added L10: 10 uH, passives:INDUCTOR0603
- added L9: 15 nH, passives:INDUCTOR0402
- added LED1: LED0603, leds:LED0603
- added R1, R2, R3: 10 K, rcl:R-US_R0603
- added R4, R5, R6, R7: (no value), passives:RESISTOR0603_RES
- added U$1: QT1070, QT1070:QT1070
- added U3: NRF51822QF, chips:NRF51822QF
- added U4: MCP73831, SparkFun-PowerIC:MCP73831
- added X2: (no value), crystals:TXC-8Y
- added X3: ABS05-32.768KHZ-9-T, crystals:ABS05-32.768KHZ-9-T
- C1, C2: value 12 pF -> (none); device rcl:C-USC0402 -> passives:CAPACITOR0603_CAP
- C3: value 2.2 nF -> (none); device rcl:C-USC0402 -> passives:CAPACITOR0603_CAP
Connections:
- removed net N$10: L4.1, U2.DCC
- removed net N$11: L4.2, L5.2
- removed net N$13: C2.1, U2.XC1, X1.2
- removed net N$5: C5.1, L1.2, U2.ANT2
- removed net N$6: C3.1, L2.1, U2.VDD_PA
- removed net N$7: C4.1, C5.2, L3.1
- removed net N$8: C6.1, L3.2
- removed net XC2: C1.1, U2.XC2, X1.1
- new net GNDIO: C13.2, C14.2, C15.2, C16.2, U1.COM2, U1.GND, U1.GNDIO, U1.PIN10, U1.PIN15, U1.PIN16
- new net I2C_ADDR_SEL: U1.COM3
- new net INT: U1.INT
- new net N$12: U1.PS0, U1.PS1
- new net N$14: L10.2, U3.DCC
- new net N$15: L10.1, L9.2
- new net N$16: C27.1, C30.1, L9.1, U3.AVDD
- new net N$17: R2.1, U1.COM0
- new net N$18: R3.1, U1.NBOOT_LOAD_PIN
- new net N$19: R4.2, U3.SWDIO/!RESET
- new net N$20: C20.1, U3.XC2, X2.2
- new net N$21: B1.ANT1, U3.ANT1
- new net N$22: B1.ANT2, U3.ANT2
- new net N$23: B1.VDD_PA, C21.1, U3.VDD_PA
- new net N$24: A1.ANTENNA, B1.SE, C24.1
- new net N$25: C28.1, U3.DEC2
- new net N$26: C22.1, U3.DEC1
- new net N$27: C17.1, U3.P26/AIN0/XL2, X3.1
- new net N$28: C18.1, U3.P27/AIN1/XL1, X3.2
- new net N$29: C19.1, U3.XC1, X2.1
- new net N$30: R5.2, U3.SWDCLK
- new net N$38: C1.1, J1.+5V, R6.2, U4.VIN
- new net SCL: R1.1, U1.COM1
- net GND: now also B1.GND, C17.2, C18.2, C19.2, C20.2, C21.2, C22.2, C24.2, C25.2, C27.2, C28.2, C29.2, C3.2, C30.2, J1.GND, R4.1, R5.1, R7.1, U3.GND, U4.VSS; no longer C4.2, C6.2, U1.GND, U1.GNDIO, U2.VSS1, U2.VSS2, U2.VSS3
- net N$1: now also C2.1, C3.1, U4.VBAT; no longer C10.2, C11.2, C12.2, C3.2, C7.2, C8.2, C9.2
- net N$2: now also LED1.ANODE, R6.1; no longer L1.1, L2.2, U2.ANT1
- net N$3: now also LED1.CATHODE, U4.STAT; no longer C8.1, U2.DEC1
- net N$4: now also R7.2, U4.PROG; no longer C10.1, U2.DEC2
- net N$9: now also C13.1
- net VCC: now also C25.1, C29.1, U3.VDD; no longer C11.1, C12.1, C7.1, C9.1, L5.1, U2.AVDD1, U2.AVDD2, U2.VDD1, U2.VDD2
- net VDD: now also C14.1, C15.1, C16.1, R1.2, R2.2, R3.2
