File: hardware/glove.sch (EAGLE design)
At the start: 84 parts, among them J1 TC2030-JLINK-NL, J2 MICRO_USB_B_JST_MC5BR3-M404-4S, P1 DMP1045U, U1 NRF51822QF, U2 BNO055, U3 AT42QT1070, U4 MCP73831, U5 LP3855EMP-ADJ, X1 ABS05-32.768KHZ-9-T

Commit message: Need to finish silkscreen
Parts:
- C17: value (none) -> 100 nF
- R7: value (none) -> 47 k
Connections:
- removed net INT: U2.INT
- removed net N$17: R8.1, U3.!CHANGE
- new net !CHANGE: R8.1, U1.P16, U3.!CHANGE
Other:
- moved on the sheet: R7, R8
Changed lines of the file:
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@@
 <?xml version="1.0" encoding="utf-8"?>
 <!DOCTYPE eagle SYSTEM "eagle.dtd">
-<eagle version="7.6.0">
+<eagle version="6.6.0">
 <drawing>
 <settings>
@@
 <part name="GND17" library="supply1" deviceset="GND" device=""/>
 <part name="P+6" library="supply1" deviceset="VCC" device=""/>
-<part name="R7" library="passives" deviceset="RESISTOR" device="0603_RES"/>
+<part name="R7" library="passives" deviceset="RESISTOR" device="0603_RES" value="47 k"/>
 <part name="R8" library="passives" deviceset="RESISTOR" device="0603_RES" value="47 k"/>
 <part name="R11" library="passives" deviceset="RESISTOR" device="0603_RES" value="10 k"/>
@@
 <part name="R12" library="passives" deviceset="RESISTOR" device="0603_RES" value="10 k"/>
 <part name="R10" library="passives" deviceset="RESISTOR" device="0603_RES" value="10 k"/>
-<part name="C17" library="passives" deviceset="CAPACITOR" device="0603_CAP"/>
+<part name="C17" library="passives" deviceset="CAPACITOR" device="0603_CAP" value="100 nF"/>
 <part name="P+5" library="supply1" deviceset="VCC" device=""/>
 <part name="LED14" library="leds" deviceset="LED" device="0603"/>
@@
 </segment>
 </net>
+<net name="!CHANGE" class="0">
+<segment>
+<pinref part="U1" gate="G$1" pin="P16"/>
+<wire x1="22.86" y1="27.94" x2="30.48" y2="27.94" width="0.1524" layer="91"/>
+<label x="30.48" y="27.94" size="1.778" layer="95"/>
+</segment>
+</net>
 </nets>
 </sheet>
@@
 </segment>
 </net>
-<net name="INT" class="0">
-<segment>
-<pinref part="U2" gate="G$1" pin="INT"/>
-<wire x1="20.32" y1="2.54" x2="25.4" y2="2.54" width="0.1524" layer="91"/>
-<label x="25.4" y="2.54" size="1.778" layer="95"/>
-</segment>
-</net>
 <net name="SDA" class="0">
 <segment>
@@
 <instance part="GND17" gate="1" x="55.88" y="25.4"/>
 <instance part="P+6" gate="VCC" x="55.88" y="83.82"/>
-<instance part="R7" gate="G$1" x="7.62" y="66.04" rot="R90"/>
-<instance part="R8" gate="G$1" x="15.24" y="66.04" rot="R90"/>
+<instance part="R7" gate="G$1" x="7.62" y="63.5" rot="R90"/>
+<instance part="R8" gate="G$1" x="22.86" y="63.5" rot="R90"/>
 <instance part="R11" gate="G$1" x="86.36" y="55.88" rot="R180"/>
 <instance part="R9" gate="G$1" x="78.74" y="53.34" rot="R180"/>
@@
 <junction x="55.88" y="78.74"/>
 <pinref part="R7" gate="G$1" pin="2"/>
-<wire x1="15.24" y1="78.74" x2="55.88" y2="78.74" width="0.1524" layer="91"/>
-<wire x1="15.24" y1="78.74" x2="7.62" y2="78.74" width="0.1524" layer="91"/>
-<wire x1="7.62" y1="78.74" x2="7.62" y2="68.58" width="0.1524" layer="91"/>
+<wire x1="22.86" y1="78.74" x2="55.88" y2="78.74" width="0.1524" layer="91"/>
+<wire x1="22.86" y1="78.74" x2="7.62" y2="78.74" width="0.1524" layer="91"/>
+<wire x1="7.62" y1="78.74" x2="7.62" y2="66.04" width="0.1524" layer="91"/>
 <pinref part="R8" gate="G$1" pin="2"/>
-<wire x1="15.24" y1="68.58" x2="15.24" y2="78.74" width="0.1524" layer="91"/>
-<junction x="15.24" y="78.74"/>
+<wire x1="22.86" y1="66.04" x2="22.86" y2="78.74" width="0.1524" layer="91"/>
+<junction x="22.86" y="78.74"/>
 <pinref part="U3" gate="G$1" pin="VDD"/>
 </segment>
@@
 </segment>
 </net>
-<net name="N$17" class="0">
+<net name="!CHANGE" class="0">
 <segment>
 <pinref part="R8" gate="G$1" pin="1"/>
-<wire x1="15.24" y1="60.96" x2="15.24" y2="53.34" width="0.1524" layer="91"/>
-<wire x1="15.24" y1="53.34" x2="38.1" y2="53.34" width="0.1524" layer="91"/>
+<wire x1="22.86" y1="58.42" x2="22.86" y2="53.34" width="0.1524" layer="91"/>
+<wire x1="22.86" y1="53.34" x2="38.1" y2="53.34" width="0.1524" layer="91"/>
 <pinref part="U3" gate="G$1" pin="!CHANGE"/>
+<wire x1="22.86" y1="53.34" x2="17.78" y2="53.34" width="0.1524" layer="91"/>
+<junction x="22.86" y="53.34"/>
+<label x="10.16" y="53.34" size="1.778" layer="95"/>
 </segment>
 </net>
@@
 <segment>
 <pinref part="R7" gate="G$1" pin="1"/>
-<wire x1="7.62" y1="60.96" x2="7.62" y2="48.26" width="0.1524" layer="91"/>
+<wire x1="7.62" y1="58.42" x2="7.62" y2="48.26" width="0.1524" layer="91"/>
 <wire x1="7.62" y1="48.26" x2="38.1" y2="48.26" width="0.1524" layer="91"/>
 <pinref part="U3" gate="G$1" pin="!RESET"/>
