File: hardware/glove.sch (EAGLE design)
At the start: 90 parts, among them J1 TC2030-JLINK-NL, J2 MICRO_USB_B_JST_MC5BR3-M404-4S, P1 DMP1045U, T0 WIREPAD1,6/0,8, T1 WIREPAD1,6/0,8, T2 WIREPAD1,6/0,8, T3 WIREPAD1,6/0,8, U1 NRF51822QF, U2 BNO055, U3 AT42QT1070, U4 MCP73831, U5 LP3855EMP-ADJ, X1 ABS05-32.768KHZ-9-T

Commit message: turns out they're not quite done...damn
Parts:
- removed R7: 150, passives:RESISTOR0603_RES
- J1: value TC2030-JLINK-NL -> TC2030-JLINK-L; device connector:TC2030-JLINK-NL -> connector:TC2030-JLINK-L
Connections:
- net GND: no longer R7.1
- net N$19: no longer R7.2
Changed lines of the file:
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@@
 <?xml version="1.0" encoding="utf-8"?>
 <!DOCTYPE eagle SYSTEM "eagle.dtd">
-<eagle version="6.6.0">
+<eagle version="7.6.0">
 <drawing>
 <settings>
@@
 <part name="P+1" library="supply1" deviceset="VCC" device=""/>
 <part name="GND9" library="supply1" deviceset="GND" device=""/>
-<part name="GND8" library="supply1" deviceset="GND" device=""/>
-<part name="R7" library="passives" deviceset="RESISTOR" device="0603_RES" value="150"/>
 <part name="R8" library="passives" deviceset="RESISTOR" device="0603_RES" value="12 k"/>
 <part name="U4" library="SparkFun-PowerIC" deviceset="MCP73831" device=""/>
@@
 <part name="P+3" library="supply1" deviceset="VCC" device=""/>
 <part name="GND6" library="supply1" deviceset="GND" device=""/>
-<part name="J1" library="connector" deviceset="TC2030-JLINK" device="-NL"/>
+<part name="J1" library="connector" deviceset="TC2030-JLINK" device="-L" value="TC2030-JLINK-L"/>
 <part name="R2" library="passives" deviceset="RESISTOR" device="0603_RES" value="1 k"/>
 <part name="P+4" library="supply1" deviceset="VCC" device=""/>
@@
 <instance part="P+1" gate="VCC" x="-2.54" y="76.2"/>
 <instance part="GND9" gate="1" x="-33.02" y="-58.42"/>
-<instance part="GND8" gate="1" x="-48.26" y="-58.42"/>
-<instance part="R7" gate="G$1" x="-48.26" y="-35.56" rot="R90"/>
 <instance part="R8" gate="G$1" x="-33.02" y="-35.56" rot="R90"/>
 <instance part="LED2" gate="G$1" x="-73.66" y="-5.08" rot="R270"/>
@@
 </segment>
 <segment>
-<pinref part="R7" gate="G$1" pin="1"/>
-<pinref part="GND8" gate="1" pin="GND"/>
-<wire x1="-48.26" y1="-40.64" x2="-48.26" y2="-55.88" width="0.1524" layer="91"/>
-</segment>
-<segment>
 <pinref part="GND6" gate="1" pin="GND"/>
 <wire x1="-86.36" y1="-33.02" x2="-91.44" y2="-33.02" width="0.1524" layer="91"/>
@@
 <segment>
 <pinref part="U1" gate="G$1" pin="SWDIO/!RESET"/>
-<pinref part="R7" gate="G$1" pin="2"/>
-<wire x1="-22.86" y1="-22.86" x2="-48.26" y2="-22.86" width="0.1524" layer="91"/>
-<wire x1="-48.26" y1="-22.86" x2="-48.26" y2="-33.02" width="0.1524" layer="91"/>
-<wire x1="-60.96" y1="-22.86" x2="-48.26" y2="-22.86" width="0.1524" layer="91"/>
-<junction x="-48.26" y="-22.86"/>
+<wire x1="-22.86" y1="-22.86" x2="-60.96" y2="-22.86" width="0.1524" layer="91"/>
 <pinref part="J1" gate="G$1" pin="SWDIO"/>
 </segment>

Commit message: Likely Ready to Order
Parts:
- removed R25: 20k, passives:RESISTOR0603_RES
- added R7: 12 k, passives:RESISTOR0603_RES
- R11: value 47 k -> 10 k
- R15: value 10 k -> 100k
- R16: value 100k -> 470
- R17: value 470 -> 2 k
- R18: value 2 k -> 250
- R19: value 250 -> 440
- R20: value 440 -> 250
- R21: value 250 -> 20k
- R8: value 12 k -> 10 k
- R9: value 10 k -> 47 k
Connections:
- net !CHANGE: now also R10.1; no longer R11.1
- net FLEX0: now also R21.1; no longer R22.1
- net FLEX1: now also R22.1; no longer R23.1
- net FLEX2: now also R23.1; no longer R24.1
- net FLEX3: now also R24.1; no longer R25.1
- net GND: now also R15.1, R17.1, R18.2, R20.1, R21.2, R7.1; no longer R16.1, R18.1, R19.2, R21.1, R25.2, R8.1
- net N$17: now also R20.2; no longer R21.2
- net N$18: now also R8.1; no longer R9.1
- net N$2: now also R16.1; no longer R17.1
- net N$30: now also R7.2; no longer R8.2
- net N$31: now also R11.2; no longer R12.2
- net N$32: now also R11.1; no longer R12.1
- net N$33: now also R12.2; no longer R13.2
- net N$34: now also R12.1; no longer R13.1
- net N$35: now also R13.2; no longer R14.2
- net N$36: now also R13.1; no longer R14.1
- net N$37: now also R14.2; no longer R15.2
- net N$38: now also R15.2; no longer R17.2
- net N$39: now also R14.1; no longer R15.1
- net N$4: now also R17.2; no longer R18.2
- net N$40: now also R9.1; no longer R10.1
- net N$7: now also R18.1, R19.2; no longer R19.1, R20.2
- net VCC: now also R19.1, R8.2; no longer R11.2, R20.1
Other:
- moved on the sheet: R10, R11, R12, R13, R14, R16, R17, R18, R19, R20, R22, R23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
