File: hardware/glove.sch (EAGLE design)
At the start: 89 parts, among them J1 TC2030-JLINK-L, J2 MICRO_USB_B_JST_MC5BR3-M404-4S, P1 DMP1045U, T0 WIREPAD1,6/0,8, T1 WIREPAD1,6/0,8, T2 WIREPAD1,6/0,8, T3 WIREPAD1,6/0,8, U1 NRF51822QF, U2 BNO055, U3 AT42QT1070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

Commit message: Added Gerber Files
Parts:
- R18: value 250 -> 5.6 k
- R19: value 440 -> 10 k
- renumbered P1 to Q1
Changed lines of the file:
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@@
 <part name="U5" library="LP3855EMP-ADJ" deviceset="LP3855EMP-ADJ" device=""/>
 <part name="C21" library="passives" deviceset="CAPACITOR" device="0603_CAP" value="8 nF"/>
-<part name="R19" library="passives" deviceset="RESISTOR" device="0603_RES" value="440"/>
-<part name="R18" library="passives" deviceset="RESISTOR" device="0603_RES" value="250"/>
+<part name="R19" library="passives" deviceset="RESISTOR" device="0603_RES" value="10 k"/>
+<part name="R18" library="passives" deviceset="RESISTOR" device="0603_RES" value="5.6 k"/>
 <part name="C22" library="passives" deviceset="CAPACITOR" device="0603_CAP" value="10 uF"/>
 <part name="C23" library="passives" deviceset="CAPACITOR" device="0603_CAP" value="10 uF"/>
@@
 <part name="GND18" library="supply1" deviceset="GND" device=""/>
 <part name="R15" library="passives" deviceset="RESISTOR" device="0603_RES" value="100k"/>
-<part name="P1" library="load_balance" deviceset="DMP1045U" device=""/>
+<part name="Q1" library="load_balance" deviceset="DMP1045U" device=""/>
 <part name="D1" library="load_balance" deviceset="B130LAW" device=""/>
 <part name="SPI+" library="wirepad" deviceset="WIREPAD" device="1,6/0,9" value="WIREPAD1,6/0,9"/>
@@
 <instance part="GND18" gate="1" x="111.76" y="40.64" rot="R180"/>
 <instance part="R15" gate="G$1" x="91.44" y="33.02" rot="R180"/>
-<instance part="P1" gate="G$1" x="60.96" y="25.4" rot="MR270"/>
+<instance part="Q1" gate="G$1" x="60.96" y="25.4" rot="MR270"/>
 <instance part="D1" gate="G$1" x="83.82" y="17.78" rot="R270"/>
 <instance part="R20" gate="G$1" x="10.16" y="-35.56" rot="R90"/>
@@
 <junction x="-50.8" y="20.32"/>
 <wire x1="-40.64" y1="20.32" x2="-40.64" y2="33.02" width="0.1524" layer="91"/>
-<pinref part="P1" gate="G$1" pin="GATE"/>
+<pinref part="Q1" gate="G$1" pin="GATE"/>
 <wire x1="-40.64" y1="33.02" x2="60.96" y2="33.02" width="0.1524" layer="91"/>
 <pinref part="R15" gate="G$1" pin="2"/>
@@
 <wire x1="101.6" y1="15.24" x2="101.6" y2="22.86" width="0.1524" layer="91"/>
 <junction x="101.6" y="22.86"/>
-<pinref part="P1" gate="G$1" pin="SOURCE"/>
+<pinref part="Q1" gate="G$1" pin="SOURCE"/>
 <wire x1="71.12" y1="20.32" x2="76.2" y2="20.32" width="0.1524" layer="91"/>
 <wire x1="76.2" y1="20.32" x2="76.2" y2="15.24" width="0.1524" layer="91"/>
@@
 <pinref part="U4" gate="G$1" pin="VBAT"/>
 <wire x1="12.7" y1="20.32" x2="40.64" y2="20.32" width="0.1524" layer="91"/>
-<pinref part="P1" gate="G$1" pin="DRAIN"/>
+<pinref part="Q1" gate="G$1" pin="DRAIN"/>
 <wire x1="40.64" y1="20.32" x2="48.26" y2="20.32" width="0.1524" layer="91"/>
 <junction x="40.64" y="20.32"/>
