File: hardware/glove.brd (EAGLE design)
At the start: 50.8 x 36.8 mm, 90 parts, among them J1 TC2030-JLINK-L, J2 MICRO_USB_B_JST_MC5BR3-M404-4S, P1 DMP1045U, T0 WIREPAD1,6/0,8, T1 WIREPAD1,6/0,8, T2 WIREPAD1,6/0,8, T3 WIREPAD1,6/0,8, U1 NRF51822QF, U2 BNO055, U3 AT42QT1070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

Commit message: Likely Ready to Order
Parts:
- removed R25: 20k, passives:0603-RES
- added R7: 12 k, passives:0603-RES
- R11: value 47 k -> 10 k
- R15: value 10 k -> 100k
- R16: value 100k -> 470
- R17: value 470 -> 2 k
- R18: value 2 k -> 250
- R19: value 250 -> 440
- R20: value 440 -> 250
- R21: value 250 -> 20k
- R8: value 12 k -> 10 k
- R9: value 10 k -> 47 k
- moved R8 39.7 mm to (12.7, 29.6), turned to 270 degrees
- moved R15 38.1 mm to (6.35, 8.89), turned to 90 degrees
- moved R9 24.2 mm to (36.4, 24.8)
- moved R20 15.0 mm to (21.3, 3.48), turned to 90 degrees
- moved R11 12.6 mm to (48.3, 27.9)
- moved R16 10.9 mm to (12.7, 17.8), turned to 180 degrees
- moved R17 10.9 mm to (19.4, 9.19), turned to 90 degrees
- moved R18 8.75 mm to (17.8, 17.8), turned to 270 degrees
- moved R10 4.88 mm to (38.2, 20.3)
- moved R13 3.81 mm to (41.9, 27.9)
- moved R21 2.95 mm to (23.5, 1.47), turned to 0 degrees
- moved R24 2.59 mm to (31.2, 1.50)
- moved R22 2.54 mm to (26.0, 1.50)
- moved R12 2.54 mm to (45.7, 27.9)
- moved R14 2.54 mm to (39.4, 27.9)
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Connections:
- net !CHANGE: now also R10.1; no longer R11.1
- net FLEX0: now also R21.1; no longer R22.1
- net FLEX1: now also R22.1; no longer R23.1
- net FLEX2: now also R23.1; no longer R24.1
- net FLEX3: now also R24.1; no longer R25.1
- net GND: now also R15.1, R17.1, R18.2, R20.1, R21.2, R7.1; no longer R16.1, R18.1, R19.2, R21.1, R25.2, R8.1
- net N$17: now also R20.2; no longer R21.2
- net N$18: now also R8.1; no longer R9.1
- net N$2: now also R16.1; no longer R17.1
- net N$30: now also R7.2; no longer R8.2
- net N$31: now also R11.2; no longer R12.2
- net N$32: now also R11.1; no longer R12.1
- net N$33: now also R12.2; no longer R13.2
- net N$34: now also R12.1; no longer R13.1
- net N$35: now also R13.2; no longer R14.2
- net N$36: now also R13.1; no longer R14.1
- net N$37: now also R14.2; no longer R15.2
- net N$38: now also R15.2; no longer R17.2
- net N$39: now also R14.1; no longer R15.1
- net N$4: now also R17.2; no longer R18.2
- net N$40: now also R9.1; no longer R10.1
- net N$7: now also R18.1, R19.2; no longer R19.1, R20.2
- net VCC: now also R19.1, R8.2; no longer R11.2, R20.1
Routing:
- net SDA: track 63.4 -> 67.0 mm
- net GND: track 36.3 -> 34.5 mm, vias 28 -> 32
- net VCC: track 160.3 -> 161.8 mm
- net N$43: track 18.1 -> 19.0 mm
- net N$12: track 13.2 -> 13.7 mm

Commit message: Added Gerber Files
Parts:
- R18: value 250 -> 5.6 k
- R19: value 440 -> 10 k
- moved LED2 0.53 mm to (39.9, 5.59)
- moved R2 0.51 mm to (41.4, 7.44)
- renumbered P1 to Q1
